Commit message: session4

File: session3/johny_description/urdf/johny.urdf (robot description, URDF)
Before this commit: robot johny, 5 links, 4 joints
Links:
- removed link sphere_link
- added link caster_wheel_link, mass 0.5; collision sphere radius=0.05; visual sphere radius=0.05
- link base_link: mass None -> 5; geometry collision box size=0.6 0.4 0.2; visual box size=0.6 0.4 0.2
- link left_wheel_link: mass None -> 1; geometry collision cylinder length=0.05 radius=0.1; visual cylinder length=0.05 radius=0.1
- link right_wheel_link: mass None -> 1; geometry collision cylinder length=0.05 radius=0.1; visual cylinder length=0.05 radius=0.1
Joints:
- removed joint base_sphere_joint
- added joint base_caster_wheel_joint: type fixed, parent base_link, child caster_wheel_link, origin xyz=0.2 0 -0.15 rpy=0 0 0
